File: HVPS/HVPS.sch (KiCad schematic (older format))
At the start: 9 parts, among them Q1 2SD2470, SW1 MSS22D18D, T1 Flash XFMR

Commit message: Add files via upload
Parts:
- C1: value 2.2uF 250v -> .22uF 250v
Changed lines of the file:
@@
 P 4450 3050
 F 0 "C1" H 4565 3096 50  0000 L CNN
-F 1 "2.2uF 250v" H 4565 3005 50  0000 L CNN
+F 1 ".22uF 250v" H 4565 3005 50  0000 L CNN
 F 2 "Capacitor_SMD:C_1206_3216Metric_Pad1.42x1.75mm_HandSolder" H 4488 2900 50  0001 C CNN
 F 3 "~" H 4450 3050 50  0001 C CNN
